Commit message: gazebo fixed with not absolute path

File: champ_description/urdf/champ.urdf (robot description, URDF)
Before this commit: robot champ, 29 links, 28 joints
Links:
- link base_link: geometry collision mesh filename=file:///home/luqman/dogbot_ws/src/champ/champ_description/m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 scale=0.001 0.001 0.001; visual mesh filename=file:///home/luqman/dogbot_ws/src/champ/champ_description/m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 scale=0.001 0.001 0.001
- link camera_link: geometry collision mesh filename=file:///home/luqman/dogbot_ws/src/champ/champ_description/m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; visual mesh filename=file:///home/luqman/dogbot_ws/src/champ/champ_description/m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
- link hokuyo_frame: geometry collision box size=0.058 0.058 0.087; visual mesh filename=file:///home/luqman/dogbot_ws/src/champ/champ_description/m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
- link lf_hip_link: geometry collision mesh filename=file:///home/luqman/dogbot_ws/src/champ/champ_description/m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 scale=0.001 0.001 0.001; visual mesh filename=file:///home/luqman/dogbot_ws/src/champ/champ_description/m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 scale=0.001 0.001 0.001
- link lf_lower_leg_link: geometry collision mesh filename=file:///home/luqman/dogbot_ws/src/champ/champ_description/m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 scale=0.001 0.001 0.001; visual mesh filename=file:///home/luqman/dogbot_ws/src/champ/champ_description/m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 scale=0.001 0.001 0.001
- link lf_upper_leg_link: geometry collision mesh filename=file:///home/luqman/dogbot_ws/src/champ/champ_description/m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 scale=0.001 0.001 0.001; visual mesh filename=file:///home/luqman/dogbot_ws/src/champ/champ_description/m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 scale=0.001 0.001 0.001
- link lh_hip_link: geometry collision mesh filename=file:///home/luqman/dogbot_ws/src/champ/champ_description/m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 scale=0.001 0.001 0.001; visual mesh filename=file:///home/luqman/dogbot_ws/src/champ/champ_description/m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 scale=0.001 0.001 0.001
- link lh_lower_leg_link: geometry collision mesh filename=file:///home/luqman/dogbot_ws/src/champ/champ_description/m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 scale=0.001 0.001 0.001; visual mesh filename=file:///home/luqman/dogbot_ws/src/champ/champ_description/m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 scale=0.001 0.001 0.001
- link lh_upper_leg_link: geometry collision mesh filename=file:///home/luqman/dogbot_ws/src/champ/champ_description/m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 scale=0.001 0.001 0.001; visual mesh filename=file:///home/luqman/dogbot_ws/src/champ/champ_description/m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 scale=0.001 0.001 0.001
- link rf_hip_link: geometry collision mesh filename=file:///home/luqman/dogbot_ws/src/champ/champ_description/m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 scale=0.001 0.001 0.001; visual mesh filename=file:///home/luqman/dogbot_ws/src/champ/champ_description/m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 scale=0.001 0.001 0.001
- link rf_lower_leg_link: geometry collision mesh filename=file:///home/luqman/dogbot_ws/src/champ/champ_description/m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 scale=0.001 0.001 0.001; visual mesh filename=file:///home/luqman/dogbot_ws/src/champ/champ_description/m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 scale=0.001 0.001 0.001
- link rf_upper_leg_link: geometry collision mesh filename=file:///home/luqman/dogbot_ws/src/champ/champ_description/m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 scale=0.001 0.001 0.001; visual mesh filename=file:///home/luqman/dogbot_ws/src/champ/champ_description/m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 scale=0.001 0.001 0.001
- link rh_hip_link: geometry collision mesh filename=file:///home/luqman/dogbot_ws/src/champ/champ_description/m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 scale=0.001 0.001 0.001; visual mesh filename=file:///home/luqman/dogbot_ws/src/champ/champ_description/m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 scale=0.001 0.001 0.001
- link rh_lower_leg_link: geometry collision mesh filename=file:///home/luqman/dogbot_ws/src/champ/champ_description/m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 scale=0.001 0.001 0.001; visual mesh filename=file:///home/luqman/dogbot_ws/src/champ/champ_description/m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 scale=0.001 0.001 0.001
- link rh_upper_leg_link: geometry collision mesh filename=file:///home/luqman/dogbot_ws/src/champ/champ_description/m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 scale=0.001 0.001 0.001; visual mesh filename=file:///home/luqman/dogbot_ws/src/champ/champ_description/m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 scale=0.001 0.001 0.001
